File: arcboard-stm32.kicad_sch (KiCad schematic)
At the start: 1 part, among them U1 STM32F405RGT6

Commit message: savegame jul23
Parts:
- removed U1: STM32F405RGT6, footprint:LQFP-64_L10.0-W10.0-P0.50-LS12.0-BL, symbol kicad-libraries:STM32F405RGT6
- added C1, C12, C5, C7, C8, C9: 100nf, Capacitor_SMD:C_0402_1005Metric, symbol Device:C_Small
- added C10: 4.7uf, Capacitor_SMD:C_0402_1005Metric, symbol Device:C_Small
- added C13, C27: 1u, kicad-libraries:C0402, symbol Device:C
- added C15: 1u, kicad-libraries:C0402, symbol ct-kicad:CL31B105KBHNNNE
- added C18, C19: 100nf, kicad-libraries:C0402, symbol ct-kicad:CL05B104KO5NNNC
- added C2, C4: 2.2uf, Capacitor_SMD:C_0402_1005Metric, symbol Device:C_Small
- added C3, C6: 12p, Capacitor_SMD:C_0402_1005Metric, symbol Device:C_Small
- added CYBOARD-MAIN1: ECT818001569, kicad-libraries:FPC-SMD_ECT818001569, symbol kicad-python:ECT818001569
- added D2: B5817, Diode_SMD:D_SOD-323, symbol Device:D_Schottky
- added D4: SMF5_0CA_C364279, kicad-libraries:SOD-123FL_L2.8-W1.8-LS3.7-BI, symbol kicad-symbols:SMF5_0CA_C364279
- added D5, D7: USBLC6-2P6_C2827693, kicad-libraries:SOT-666-6_L1.6-W1.2-P0.50-LS1.6-BL, symbol ct-kicad:USBLC6-2P6_C2827693
- added F1: Polyfuse, kicad-libraries:F1206, symbol ct-kicad:RF1989-000
- added F3: MF-NSMF075-2, kicad-libraries:F1206, symbol kicad-symbols:MF-NSMF075-2
- added J1: Conn_01x02_Socket, Connector_PinSocket_2.54mm:PinSocket_1x02_P2.54mm_Vertical, symbol Connector:Conn_01x02_Socket
- added J13, J14, J15, J16, J3, J4, J6, J7, J8: ~, kicad-libraries:FFC-SMD_FFC05001-12SBA124W5M, symbol vik:vik-keyboard-connector
- added JP2, JP3: SolderJumper_3_Open, Jumper:SolderJumper-3_P1.3mm_Open_Pad1.0x1.5mm, symbol Jumper:SolderJumper_3_Open
- added L1: MPZ2012S101AT000, kicad-libraries:L0805, symbol kicad-symbols:MPZ2012S101AT000
- added LED-LVL1: SN74LVC1T45DRL, kicad-libraries:SOT-563_L1.6-W1.2-P0.50-LS1.6-BR, symbol Logic_LevelTranslator:SN74LVC1T45DRL
- added MOSFET1: AO3401A_C347476, kicad-libraries:SOT-23_L2.9-W1.3-P1.90-LS2.4-BR, symbol ct-kicad:AO3401A
- added R1, R11, R12, R20: 10k, Resistor_SMD:R_0402_1005Metric, symbol Device:R
- added R10, R4, R5: 5.1k, Resistor_SMD:R_0402_1005Metric, symbol Device:R
- added U1: XC6210B332MR-G, Package_TO_SOT_SMD:SOT-23-5, symbol Regulator_Linear:AP2127K-3.3
- added U2: TYPE-C-31-M-13, kicad-libraries:USB-C_SMD-TYPE-C-31-M-12, symbol kicad-libraries:TYPE-C-31-M-13
- added U3: STM32F405RGTx, Package_QFP:LQFP-64_10x10mm_P0.5mm, symbol MCU_ST_STM32F4:STM32F405RGTx
- added U4: PJ-320A, kicad-libraries:AUDIO-TH_XKB_PJ-320A, symbol kicad-libraries:PJ-320A
- added U5, U6, U7, U8, U9: BAV70S,115, kicad-libraries:SOT-363-6_L2.0-W1.3-P0.65-LS2.1-BL, symbol kicad-libraries:BAV70S,115
- added Y1: Crystal_GND24, kicad-libraries:CRYSTAL-SMD_4P-L3.2-W2.5-BL-1, symbol Device:Crystal_GND24
Connections:
- new net: J4.10 (SPI_CS), U7.2
- new net: J4.11 (MISO), U7.5
- new net: J4.7 (GP_AD1), U5.2
- new net: J4.8 (MOSI), U6.2
- new net: J4.9 (GP_AD2), U6.5
- new net: J6.10 (SPI_CS), U7.1
- new net: J6.11 (MISO), U7.4
- new net: J6.7 (GP_AD1), U5.1
- new net: J6.8 (MOSI), U6.1
- new net: J6.9 (GP_AD2), U6.4
- new net: D2.2 (A), F1.2
- new net: F3.2, L1.1
- new net: J7.7 (GP_AD1), U5.4
- new net: J8.7 (GP_AD1), U5.5
- new net: J8.10 (SPI_CS), U9.2
- new net: J8.11 (MISO), U9.5
- new net: J8.8 (MOSI), U8.2
- new net: J8.9 (GP_AD2), U8.5
- new net: J7.10 (SPI_CS), U9.1
- new net: J7.11 (MISO), U9.4
- new net: J7.8 (MOSI), U8.1
- new net: J7.9 (GP_AD2), U8.4
- new net: C2.2, U3.31 (VCAP_1)
- new net: C4.2, U3.47 (VCAP_2)
- new net: JP2.3 (B), MOSFET1.2 (S)
- new net: D4.2 (A), F3.1, MOSFET1.3 (D)
- new net: JP3.1 (A), R12.2
- new net: JP3.3 (B), R20.2
- new net +3V3: C10.2, C12.2, C15.1, C18.1, C27.1, C5.2, C7.2, C8.2, C9.2, J1.1 (Pin_1), J13.1 (3V3), J14.1 (3V3), J15.1 (3V3), J16.1 (3V3), J3.1 (3V3), LED-LVL1.1 (VCCA), LED-LVL1.5 (DIR), R20.1, U1.5 (VOUT), U3.1 (VBAT), U3.13 (VDDA), U3.19 (VDD), U3.32 (VDD), U3.48 (VDD), U3.64 (VDD)
- new net +5V: C13.1, C19.1, CYBOARD-MAIN1.13, CYBOARD-MAIN1.14, CYBOARD-MAIN1.15, CYBOARD-MAIN1.16, D2.1 (K), D5.5 (VBUS), D7.5 (VBUS), J16.6 (5V), J4.3 (SDA), J6.3 (SDA), J7.3 (SDA), J8.3 (SDA), JP2.2 (C), LED-LVL1.6 (VCCB), U1.1 (VIN), U1.3 (EN)
- new net BOOT0: J1.2 (Pin_2), R1.2, U3.60 (BOOT0)
- new net COL0: CYBOARD-MAIN1.2
- new net COL1: CYBOARD-MAIN1.20
- new net COL10: U7.3, U9.3
- new net COL2: CYBOARD-MAIN1.21
- new net COL3: CYBOARD-MAIN1.22
- new net COL4: CYBOARD-MAIN1.17
- new net COL5: CYBOARD-MAIN1.7
- new net COL6: CYBOARD-MAIN1.6, U5.3, U5.6
- new net COL7: CYBOARD-MAIN1.25, U6.6, U8.6
- new net COL8: U6.3, U8.3
- new net COL9: U7.6, U9.6
- new net ENCODER1-r1: J14.7 (GP_AD1)
- new net ENCODER1-r2: J14.9 (GP_AD2)
- new net ENCODER2-r1: J15.7 (GP_AD1)
- new net ENCODER2-r2: J15.9 (GP_AD2)
- new net ENCODER3-r1: J3.7 (GP_AD1)
- new net ENCODER3-r2: J3.9 (GP_AD2)
- new net GND: C1.2, C10.1, C12.1, C13.2, C15.2, C18.2, C19.2, C2.1, C27.2, C3.2, C4.1, C5.1, C6.2, C7.1, C8.1, C9.1, CYBOARD-MAIN1.10, CYBOARD-MAIN1.11, CYBOARD-MAIN1.26, CYBOARD-MAIN1.27, CYBOARD-MAIN1.8, CYBOARD-MAIN1.9, D4.1 (K), D5.2 (GND), D7.2 (GND), J13.2 (GND), J14.2 (GND), J15.2 (GND), J16.2 (GND), J3.2 (GND), J4.1 (3V3), J4.12 (SCLK), J4.2 (GND), J6.1 (3V3), J6.12 (SCLK), J6.2 (GND), J7.1 (3V3), J7.12 (SCLK), J7.2 (GND), J8.1 (3V3), J8.12 (SCLK), J8.2 (GND), LED-LVL1.2 (GND), MOSFET1.1 (G), R1.1, R11.1, R12.1, R4.2, R5.2, U1.2 (GND), U2.A1 (GND), U2.A12 (GND), U2.B1 (GND), U2.B12 (GND), U3.12 (VSSA), U3.18 (VSS), U3.63 (VSS), U4.5, Y1.2, Y1.4
- new net LCD1_CS: J16.10 (SPI_CS)
- new net LCD_BL: J16.11 (MISO)
- new net LCD_DC: J16.7 (GP_AD1)
- new net LCD_RST: J16.9 (GP_AD2)
- new net LED_DPAD_DI: CYBOARD-MAIN1.1
- new net LED_INDICATORS_DI: J8.4 (SCL)
- new net LED_KEYS_DI: CYBOARD-MAIN1.12, J6.4 (SCL), LED-LVL1.4 (B)
- new net LED_PADDLE1_DI: J4.5 (RGB_DO), J6.5 (RGB_DO)
- new net LED_PADDLE2_DI: J4.4 (SCL), J7.5 (RGB_DO)
- new net LED_PADDLE3_DI: J7.4 (SCL), J8.5 (RGB_DO)
- new net LED_SIG_OUTPUT: LED-LVL1.3 (A), U3.41 (PA8)
- new net NRST: C1.1, U3.7 (NRST)
- new net PH0: C3.1, U3.5 (PH0), Y1.1
- new net PH1: C6.1, U3.6 (PH1), Y1.3
- new net PMW_CS: J13.10 (SPI_CS)
- new net ROW0: CYBOARD-MAIN1.3
- new net ROW1: CYBOARD-MAIN1.4
- new net ROW2: CYBOARD-MAIN1.18
- new net ROW3: CYBOARD-MAIN1.5
- new net ROW4: CYBOARD-MAIN1.23, J4.6 (5V)
- new net ROW5: CYBOARD-MAIN1.19, J6.6 (5V), J7.6 (5V)
- new net ROW6: CYBOARD-MAIN1.24, J8.6 (5V)
- new net SERIAL_RX: D5.1 (I/O1), D5.6 (I/O1), U3.43 (PA10), U4.4
- new net SERIAL_TX: D5.3 (I/O2), D5.4 (I/O2), U3.42 (PA9), U4.3
- new net SPI1_CLK: J13.12 (SCLK), J16.12 (SCLK)
- new net SPI1_MISO: J13.11 (MISO), U3.22 (PA6)
- new net SPI1_MOSI: J13.8 (MOSI), J16.8 (MOSI), U3.23 (PA7)
- new net SPI1_SCK: U3.21 (PA5)
- new net SPLIT_HAND: JP3.2 (C)
- new net Serial_VBUS: JP2.1 (A), L1.2, U4.2
- new net SourceSinkPulldown: R4.1, R5.1, U2.A5 (CC1), U2.B5 (CC2)
- new net USB_CONN_DM: D7.1 (I/O1), D7.6 (I/O1), U2.A7 (DN1), U2.B7 (DN2), U3.44 (PA11)
- new net USB_CONN_DP: D7.3 (I/O2), D7.4 (I/O2), U2.A6 (DP1), U2.B6 (DP2), U3.45 (PA12)
- new net VBUS: F1.1, R10.2, U2.A4 (VBUS), U2.A9 (VBUS), U2.B4 (VBUS), U2.B9 (VBUS)
- new net VBUS_DETECT: R10.1, R11.2, U3.54 (PD2)
- no-connect marks 0 -> 36
Other:
- note added: "5-way switch (dpad)"
- note added: "ALL COL6"
- note added: "Cyboard flex-pcb main 25-pin connector"
- note added: "DPAD1/PAD1 COL7/8"
- note added: "DPAD1/PAD1 COL9/10"
- note added: "Encoder1 (top, back)"
- note added: "Encoder2 (top, front)"
- note added: "Encoder3 (ring)"
- note added: "LCD"
- note added: "Main-USB ESD"
- note added: "PAD2/3 COL9/10"
- note added: "PAD2/PAD3 COL7/8"
- note added: "PMW connector"
- note added: "Paddle-dpads"
- note added: "Peripheral devices"
- note added: "Power protection"
- note added: "Serial-TRRS ESD"
- note added: "Serial_VBUS"
- note added: "Split hand"
- note added: "The boot loader is located in system memory. It is used to reprogram the flash memory by using USART1 (PA9/PA10), USART3 (PC10/PC11 or PB10/PB11), CAN2 (PB5/PB13), USB OTG FS in Device mode (PA11/PA12) through DFU (device firmware upgrade)."
- note added: "VBUS detection"
- note added: "WS2818 level shifter"

Commit message: mostly there
Parts:
- added C11, C14, C16, C17: 100nf, Capacitor_SMD:C_0402_1005Metric, symbol Device:C_Small
- added C20: 4.7uf, Capacitor_SMD:C_0402_1005Metric, symbol Device:C_Small
- added H1, H2, H3, H4: MountingHole, MountingHole:MountingHole_3.2mm_M3_Pad_Via, symbol kicad-libraries:MountingHole
- added J10, J2, J5: Conn_01x02_Socket, Connector_PinSocket_1.27mm:PinSocket_1x02_P1.27mm_Vertical, symbol Connector:Conn_01x02_Socket
- added J9: Conn_01x03_Socket, Connector_PinHeader_2.54mm:PinHeader_1x03_P2.54mm_Vertical, symbol Connector:Conn_01x03_Socket
- added R2: 1k, Resistor_SMD:R_0402_1005Metric, symbol Device:R
- added REF1: SN74AHC1G14DRLR, kicad-libraries:SOT-553-5_L1.6-W1.2-P0.50-LS1.6-BL, symbol kicad-libraries:SN74AHC1G14DRLR
- added U10: 1N4148W_C81598, kicad-libraries:SOD-123F_L2.7-W1.6-LS3.8-RD, symbol kicad-libraries:1N4148W_C81598
- C1: value 100nf -> 4.7uf; footprint Capacitor_SMD:C_0402_1005Metric -> Capacitor_SMD:C_0805_2012Metric
- J1: footprint Connector_PinSocket_2.54mm:PinSocket_1x02_P2.54mm_Vertical -> Connector_PinSocket_1.27mm:PinSocket_1x02_P1.27mm_Vertical
- R1: value 10k -> 75k
Connections:
- net ENCODER1-r1 is gone; now on net ENCODER1_R1: J14.7 (GP_AD1)
- net ENCODER1-r2 is gone; now on net ENCODER1_R2: J14.9 (GP_AD2)
- net ENCODER2-r1 is gone; now on net ENCODER2_R1: J15.7 (GP_AD1)
- net ENCODER2-r2 is gone; now on net ENCODER2_R2: J15.9 (GP_AD2)
- net ENCODER3-r1 is gone; now on net ENCODER3_R1: J3.7 (GP_AD1)
- net ENCODER3-r2 is gone; now on net ENCODER3_R2: J3.9 (GP_AD2)
- net LCD1_CS is gone; now on net LCD_CS: J16.10 (SPI_CS)
- net SPI1_SCK is gone; now on net SPI1_CLK: U3.21 (PA5)
- net +3V3: now also C11.2, C17.1, J5.1 (Pin_1), REF1.5 (VCC)
- net +5V: now also C1.1, C20.2, J9.2 (Pin_2)
- net BOOT0: now also C14.1, U10.1 (K)
- net COL0: now also U3.62 (PB9)
- net COL1: now also U3.4 (PC15)
- net COL10: now also U3.50 (PA15)
- net COL11: now also U3.56 (PB4)
- net COL12: now also U3.57 (PB5)
- net COL13: now also U3.58 (PB6)
- net COL2: now also U3.3 (PC14)
- net COL3: now also U3.2 (PC13)
- net COL4: now also U3.59 (PB7)
- net COL5: now also U3.61 (PB8)
- net COL6: now also U3.55 (PB3)
- net COL7: now also U3.53 (PC12)
- net COL8: now also U3.52 (PC11)
- net COL9: now also U3.51 (PC10)
- net ENCODER1_R1: now also U3.39 (PC8)
- net ENCODER1_R2: now also U3.38 (PC7)
- net ENCODER2_R1: now also U3.37 (PC6)
- net ENCODER2_R2: now also U3.36 (PB15)
- net ENCODER3_R1: now also U3.35 (PB14)
- net ENCODER3_R2: now also U3.34 (PB13)
- net GND: now also C11.1, C14.2, C16.2, C17.2, C20.1, J2.1 (Pin_1), J9.1 (Pin_1), REF1.3 (GND)
- net LCD_BL: now also U3.28 (PB2)
- net LCD_CS: now also U3.25 (PC5)
- net LCD_DC: now also U3.26 (PB0)
- net LCD_RST: now also U3.27 (PB1)
- net LED_DPAD_DI: now also J6.4 (SCL)
- net LED_INDICATORS_DI: now also J9.3 (Pin_3)
- net LED_KEYS_DI: no longer J6.4 (SCL)
- net NRST: now also C16.1, J2.2 (Pin_2), R2.2; no longer C1.1
- net PMW_CS: now also U3.24 (PC4)
- net ROW0: now also U3.8 (PC0)
- net ROW1: now also U3.9 (PC1)
- net ROW2: now also U3.10 (PC2)
- net ROW3: now also U3.11 (PC3)
- net ROW4: now also U3.14 (PA0)
- net ROW5: now also U3.15 (PA1)
- net ROW6: now also U3.16 (PA2)
- net SPLIT_HAND: now also U3.40 (PC9)
- net USB_CONN_DM: no longer D7.1 (I/O1), U3.44 (PA11)
- net USB_CONN_DP: no longer D7.3 (I/O2), U3.45 (PA12)
- net ROW7: now reaches U3.17 (PA3)
- net SWDIO: now reaches U3.46 (PA13)
- net SWDIO: now also J10.2 (Pin_2)
- net SWCLK: now reaches U3.49 (PA14)
- net SWCLK: now also J10.1 (Pin_1)
- new net: R2.1, REF1.4 (Y)
- new net: J5.2 (Pin_2), REF1.2 (A), U10.2 (A)
- new net USB_DM: D7.1 (I/O1), U3.44 (PA11)
- new net USB_DP: D7.3 (I/O2), U3.45 (PA12)
- no-connect marks 36 -> 37
Other:
- note added: "CPU caps"
- note added: "DFU, RESET, BOOT Buttons"
- note added: "Debug"
- note added: "Dpad & paddle-dpads"
- note removed: "5-way switch (dpad)"
- note removed: "Paddle-dpads"
- moved on the sheet: C10, C12, C18, C19, C5, C7, C8, C9, J1, R1

Commit message: savegame
Parts:
- added R7, R8: 10k, Resistor_SMD:R_0402_1005Metric, symbol Device:R
- added U12, U13: AO3401A, kicad-libraries:SOT-23_L2.9-W1.3-P1.90-LS2.4-BR, symbol kicad-libraries:AO3401A
Connections:
- net +3V3: now also R7.1, R8.1, U12.3 (D); no longer C15.1, J16.1 (3V3)
- net +5V: now also U13.3 (D); no longer C1.1, C20.2, CYBOARD-MAIN1.13, CYBOARD-MAIN1.14, CYBOARD-MAIN1.15, CYBOARD-MAIN1.16, J16.6 (5V), J4.3 (SDA), J6.3 (SDA), J7.3 (SDA), J8.3 (SDA), J9.2 (Pin_2)
- net GND: now also J13.13 (PAD), J13.14 (PAD), J14.13 (PAD), J14.14 (PAD), J15.13 (PAD), J15.14 (PAD), J16.13 (PAD), J16.14 (PAD), J3.13 (PAD), J3.14 (PAD), J4.13 (PAD), J4.14 (PAD), J6.13 (PAD), J6.14 (PAD), J7.13 (PAD), J7.14 (PAD), J8.13 (PAD), J8.14 (PAD)
- net SPLIT_HAND: now also U3.33 (PB12); no longer U3.40 (PC9)
- net LCD_ON: now reaches U3.29 (PB10)
- net LCD_ON: now also R8.2, U12.1 (G)
- new net LCD_3V3: C15.1, J16.1 (3V3), U12.2 (S)
- new net RGB_5V: C1.1, C20.2, CYBOARD-MAIN1.13, CYBOARD-MAIN1.14, CYBOARD-MAIN1.15, CYBOARD-MAIN1.16, J4.3 (SDA), J6.3 (SDA), J7.3 (SDA), J8.3 (SDA), J9.2 (Pin_2), U13.2 (S)
- new net RGB_ON: R7.2, U13.1 (G), U3.40 (PC9)
- no-connect marks 37 -> 38
Other:
- note added: "Crystal"
- note added: "LCD power"
- note added: "RGB power"
- moved on the sheet: R10, R11

Commit message: cleaned up routing quite a bit
Parts:
- removed J1, J2: Conn_01x02_Socket, Connector_PinSocket_1.27mm:PinSocket_1x02_P1.27mm_Vertical, symbol Connector:Conn_01x02_Socket
- added JP1, JP4: SolderJumper_3_Open, Jumper:SolderJumper-3_P1.3mm_Open_RoundedPad1.0x1.5mm, symbol Jumper:SolderJumper_3_Open
- added U11, U14, U15: TS-1187A-B-A-B, kicad-libraries:SW-SMD_4P-L5.1-W5.1-P3.70-LS6.5-TL_H1.5, symbol kicad-libraries:TS-1187A-B-A-B
- J5: footprint Connector_PinSocket_1.27mm:PinSocket_1x02_P1.27mm_Vertical -> Connector_PinSocket_2.54mm:PinSocket_1x02_P2.54mm_Vertical
Connections:
- net +3V3: now also U11.1 (A), U11.2 (B), U15.1 (A), U15.2 (B)
- net BOOT0: now also U11.3 (C), U11.4 (D)
- net COL0: now also U3.58 (PB6); no longer U3.62 (PB9)
- net COL11: no longer U3.56 (PB4)
- net COL12: no longer U3.57 (PB5)
- net COL13: no longer U3.58 (PB6)
- net COL4: now also U3.56 (PB4); no longer U3.59 (PB7)
- net COL5: now also U3.57 (PB5); no longer U3.61 (PB8)
- net GND: now also JP1.1 (A), JP4.1 (A), U14.1 (A), U14.2 (B)
- net LCD_ON: now also JP4.3 (B); no longer U12.1 (G)
- net NRST: now also U14.3 (C), U14.4 (D)
- net RGB_ON: now also JP1.3 (B); no longer U13.1 (G)
- net ROW7: no longer U3.17 (PA3)
- net SWCLK: now also J10.2 (Pin_2); no longer J10.1 (Pin_1)
- net SWDIO: now also J10.1 (Pin_1); no longer J10.2 (Pin_2)
- net at J5.2 (Pin_2), REF1.2 (A), U10.2 (A): now also U15.3 (C), U15.4 (D)
- new net: JP4.2 (C), U12.1 (G)
- new net: JP1.2 (C), U13.1 (G)
Other:
- moved on the sheet: R7, R8

Commit message: prepping for review
Parts:
- removed J10: Conn_01x02_Socket, Connector_PinSocket_1.27mm:PinSocket_1x02_P1.27mm_Vertical, symbol Connector:Conn_01x02_Socket
- added J2: Conn_01x04_Socket, Connector_PinSocket_1.00mm:PinSocket_1x04_P1.00mm_Vertical, symbol Connector:Conn_01x04_Socket
- C1: value 4.7uf -> 4.7uF; LCSC C1547 -> C1779
- C10, C20: value 4.7uf -> 4.7uF; footprint Capacitor_SMD:C_0402_1005Metric -> Capacitor_SMD:C_0805_2012Metric; LCSC C1547 -> C1779
- C11, C12, C14, C16, C17, C5, C7, C8, C9: value 100nf -> 100nF; LCSC C1547 -> C1525
- C13, C15, C27: value 1u -> 1uF; footprint kicad-libraries:C0402 -> Capacitor_SMD:C_0402_1005Metric
- C18, C19: value 100nf -> 100nF; footprint kicad-libraries:C0402 -> Capacitor_SMD:C_0402_1005Metric
- C2, C4: value 2.2uf -> 2.2uF; LCSC C1547 -> C12530
- H1, H2, H3, H4, J5, J9, U4: now left out of the parts list
- J13, J14, J15, J16, J3, J4, J6, J7, J8: value ~ -> FFC05001-12SBA124W5M; LCSC (none) -> C2833760
- MOSFET1: value AO3401A_C347476 -> AO3401A
- R1: value 75k -> 51k; LCSC (none) -> C25794
- R2: LCSC (none) -> C11702
- U3: LCSC (none) -> C15742
- renumbered U13 to MOSFET2, U12 to MOSFET3
Connections:
- net +3V3: now also J2.2 (Pin_2)
- net COL10: now also J6.11 (MISO), U7.4
- net COL6: now also J6.7 (GP_AD1), U5.1
- net COL7: now also J6.8 (MOSI), U6.1
- net COL8: now also J6.9 (GP_AD2), U6.4
- net COL9: now also J6.10 (SPI_CS), U7.1
- net GND: now also J2.1 (Pin_1)
- net SWCLK: now also J2.3 (Pin_3)
- net SWDIO: now also J2.4 (Pin_4)
- net SourceSinkPulldown renamed CC1-SourceSinkPulldown
- net CC1-SourceSinkPulldown: no longer R5.1, U2.B5 (CC2)
- new net CC2-SourceSinkPulldown: R5.1, U2.B5 (CC2)
Other:
- note added: "Encoders"
- note added: "MCU; power, timing, & boot"
- note added: "Main USB"
- note added: "Other"
- note added: "Power - 3V3"
- note added: "RGB LED chain output"
- note added: "RGB LED power"
- note added: "RGB LEDs"
- note added: "ROW2COL - Keys, dpads"
- note added: "SPI devices"
- note added: "Serial TRRS"
- note added: "USB-C connector"
- note added: "VBUS power protection"
- note removed: "Peripheral devices"
- note removed: "Power protection"
- note removed: "RGB power"
- moved on the sheet: C1, C10, C11, C12, C13, C14, C15, C16, C17, C18, C19, C2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

Commit message: before removal of usb port
Parts:
- removed C16: 100nF, Capacitor_SMD:C_0402_1005Metric, symbol Device:C_Small
- removed R1: 51k, Resistor_SMD:R_0402_1005Metric, symbol Device:R
- removed R2: 1k, Resistor_SMD:R_0402_1005Metric, symbol Device:R
- removed REF1: SN74AHC1G14DRLR, kicad-libraries:SOT-553-5_L1.6-W1.2-P0.50-LS1.6-BL, symbol kicad-libraries:SN74AHC1G14DRLR
- removed U11, U14: TS-1187A-B-A-B, kicad-libraries:SW-SMD_4P-L5.1-W5.1-P3.70-LS6.5-TL_H1.5, symbol kicad-libraries:TS-1187A-B-A-B
- removed U4: PJ-320A, kicad-libraries:AUDIO-TH_XKB_PJ-320A, symbol kicad-libraries:PJ-320A
- added C22: CL10A106MA8NRNC, Capacitor_SMD:C_0201_0603Metric, symbol kicad-libraries:CL10A106MA8NRNC
- added J10: Conn_01x04_Socket, Connector_PinHeader_1.00mm:PinHeader_1x04_P1.00mm_Vertical, symbol Connector:Conn_01x04_Socket
- added R1: 0402WGF1004TCE, Resistor_SMD:R_0402_1005Metric, symbol kicad-libraries:0402WGF1004TCE
- added R13, R2, R3: 0402WGF1002TCE, Resistor_SMD:R_0402_1005Metric, symbol kicad-libraries:0402WGF1002TCE
- added R14: 0402WGF1000TCE, Resistor_SMD:R_0402_1005Metric, symbol kicad-libraries:0402WGF1000TCE
- added R15: 0402WGF1001TCE, Resistor_SMD:R_0402_1005Metric, symbol kicad-libraries:0402WGF1001TCE
- added R6: 0603WAF3303T5E, Resistor_SMD:R_0201_0603Metric, symbol kicad-libraries:0603WAF3303T5E
- added R9: 0402WGF1003TCE, Resistor_SMD:R_0402_1005Metric, symbol kicad-libraries:0402WGF1003TCE
- added U11: W25Q16JVSSIQTR, kicad-libraries:SOIC-8_L5.3-W5.3-P1.27-LS8.0-BL, symbol kicad-libraries:W25Q16JVSSIQTR
- added U12: TYPE-C-31-M-13, kicad-libraries:USB-C_SMD-TYPE-C-31-M-12, symbol kicad-libraries:TYPE-C-31-M-13
- added U13, U4: 2N7002, kicad-libraries:SOT-23-3_L2.9-W1.3-P1.90-LS2.4-BR, symbol kicad-libraries:2N7002
Connections:
- net +3V3: now also C14.2, J10.3 (Pin_3), U11.3 (IO2), U11.7 (IO3), U11.8 (VCC); no longer C17.1
- net BOOT0: now also C22.1, J10.4 (Pin_4), R1.1, R13.1, R6.2; no longer C14.1, U10.1 (K)
- net GND: now also C14.1, C17.1, C22.2, J10.1 (Pin_1), R1.2, R3.2, R9.2, U11.4 (GND), U12.A1 (GND), U12.A12 (GND), U12.B1 (GND), U12.B12 (GND), U13.2 (S), U4.2 (S); no longer C14.2, C17.2
- net NRST: now also C17.2, J10.2 (Pin_2), R14.2
- net SPI1_CLK: now also U11.6 (CLK)
- net SPI1_MISO: now also U11.2 (DO/IO1)
- net SPI1_MOSI: now also U11.5 (DI/IO0)
- net Serial_VBUS: now also U12.A4 (VBUS), U12.A9 (VBUS), U12.B4 (VBUS), U12.B9 (VBUS)
- net FLASH_CS: now reaches U3.30 (PB11)
- net FLASH_CS: now also U11.1 (/CS)
- net at J5.2 (Pin_2), U10.2 (A), U15.3 (C)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: now also R15.1
- net SERIAL_RX renamed SERIAL_CONN_RX
- net SERIAL_CONN_RX: now also U12.A6 (DP1), U12.B6 (DP2)
- net SERIAL_TX renamed SERIAL_CONN_TX
- net SERIAL_CONN_TX: now also U12.A7 (DN1), U12.B7 (DN2)
- new net: R2.2, R9.1, U4.1 (G)
- new net: R13.2, U4.3 (D)
- new net: R15.2, R3.1, U13.1 (G)
- new net: R14.1, R2.1, U13.3 (D)
- new net: R6.1, U10.1 (K)
- no-connect marks 38 -> 42
Other:
- moved on the sheet: C17, D4, D5, F3, J14, J15, J3, JP2, L1, MOSFET1, U10
